Commit message: IMU Integration

File: src/viz/urdf/topplebot.urdf (robot description, URDF)
Before this commit: robot topplebot, 2 links, 1 joints
Links:
- added link imu_link; visual sphere radius=0.02
- link base_link: geometry visual box size=0.127 0.127 0.127
Joints:
- added joint imu_joint: type fixed, parent base_link, child imu_link, origin xyz=0.0309 -0.0708 0.0536 rpy=0.61549 0.7854 1.5708

Commit message: Correct quaternion at start

File: src/viz/urdf/topplebot.urdf (robot description, URDF)
Before this commit: robot topplebot, 3 links, 2 joints
Joints:
- joint base_joint: origin xyz=0 0 0 rpy=0 0 0 -> xyz=0 0 0 rpy=-0.785398 0.6154797 -0.261799

Commit message: Working demonstration

File: src/viz/urdf/topplebot.urdf (robot description, URDF)
Before this commit: robot topplebot, 3 links, 2 joints
Links:
- removed link imu_link
- link base_link: geometry visual mesh filename=package://viz/meshes/Orientation_Display_Assy_01.stl scale=0.001 0.001 0.001
Joints:
- removed joint imu_joint
- joint base_joint: origin xyz=0 0 0 rpy=-0.785398 0.6154797 -0.261799 -> xyz=0 0 0 rpy=0 0 0

Commit message: Added odometry capabilites, NOT FUNCTIONAL, but is RUNNNING

File: src/viz/urdf/topplebot.urdf (robot description, URDF)
Before this commit: robot topplebot, 2 links, 1 joints
Links:
- removed link world
- added link node_0; visual box size=0.01 0.01 0.01
Joints:
- removed joint base_joint
- added joint base_link_joint: type fixed, parent node_0, child base_link, origin xyz=0 0 0 rpy=0 0 0

Commit message: Fixing URDF and correction quaternion

File: src/viz/urdf/topplebot.urdf (robot description, URDF)
Before this commit: robot topplebot, 2 links, 1 joints
Links:
- added link balancing_node, mass 0.01; visual box size=0.01 0.01 0.01
- added link world, mass 0.01; visual box size=0.01 0.01 0.01
- link node_0: mass None -> 0.01
Joints:
- added joint balancing_node_joint: type fixed, parent node_0, child balancing_node, origin xyz=0 0 0 rpy=0 0 0
- added joint world_joint: type fixed, parent world, child node_0, origin xyz=0 0 0 rpy=0 0 0

Commit message: URDF and odometry changes

File: src/viz/urdf/topplebot.urdf (robot description, URDF)
Before this commit: robot topplebot, 4 links, 3 joints
Links:
- removed link node_0
Joints:
- removed joint balancing_node_joint
- removed joint base_link_joint
- removed joint world_joint
- added joint balancing_node_to_base_link: type fixed, parent balancing_node, child base_link, origin xyz=0 0 0 rpy=0 0 0
- added joint world_to_balancing_node: type fixed, parent world, child balancing_node, origin xyz=0 0 0 rpy=0 0 0

Commit message: Adding calibration tool visual

File: src/viz/urdf/topplebot.urdf (robot description, URDF)
Before this commit: robot topplebot, 3 links, 2 joints
Links:
- link base_link: geometry visual mesh filename=package://viz/meshes/Calibration_Tool_01.stl scale=0.001 0.001 0.001

Commit message: adding balancing demo

File: src/viz/urdf/topplebot.urdf (robot description, URDF)
Before this commit: robot topplebot, 3 links, 2 joints
Links:
- link base_link: geometry visual box size=0.15 0.15 0.15

Commit message: Adding CUBEBAS viz for demo

File: src/viz/urdf/topplebot.urdf (robot description, URDF)
Before this commit: robot topplebot, 3 links, 2 joints
Links:
- link base_link: geometry visual mesh filename=package://viz/meshes/CUBEBAS.stl scale=0.001 0.001 0.001
